File: pm2008-adapter-board.kicad_sch (KiCad schematic)
At the start: 3 parts

Commit message: feat: update schematic
Parts:
- J1: renamed from J?; value (none) -> Conn_02x05_Top_Bottom
- J2: renamed from J?; value (none) -> Conn_01x04
- J3: renamed from J?; value (none) -> Conn_01x02
Connections:
- net VDD: now reaches J1.1 (Pin_1)
- net VDD: now also J1.2 (Pin_2), J2.1 (Pin_1)
- net Earth: now reaches J1.3 (Pin_3)
- net Earth: now also J1.4 (Pin_4), J2.2 (Pin_2), J3.2 (Pin_2)
- net RXD/SDA: now reaches J1.7 (Pin_7)
- net RXD/SDA: now also J2.3 (Pin_3)
- net CTL: now reaches J1.8 (Pin_8)
- net CTL: now also J3.1 (Pin_1)
- net TXD/SCL: now reaches J1.9 (Pin_9)
- net TXD/SCL: now also J2.4 (Pin_4)
- no-connect marks 0 -> 3
Other:
- moved on the sheet: J2, J3

Commit message: feat: update schematic
Changed lines of the file:
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@@
       (effects (font (size 1.27 1.27)) hide)
     )
-    (property "Value" "" (id 1) (at 98.425 81.28 0))
+    (property "Value" "VDD" (id 1) (at 98.425 81.28 0))
     (property "Footprint" "" (id 2) (at 98.425 86.36 0)
       (effects (font (size 1.27 1.27)) hide)
@@
       (effects (font (size 1.27 1.27)) hide)
     )
-    (property "Value" "" (id 1) (at 98.425 107.95 0)
+    (property "Value" "Earth" (id 1) (at 98.425 107.95 0)
       (effects (font (size 1.27 1.27)) hide)
     )
@@
     )
     (path "/7269c319-0767-4b85-898a-3b8bb1c1b467"
-      (reference "J1") (unit 1) (value "Conn_02x05_Top_Bottom") (footprint "")
+      (reference "J1") (unit 1) (value "Conn_02x05_Top_Bottom") (footprint "Connector_PinHeader_1.27mm:PinHeader_2x05_P1.27mm_Vertical")
     )
     (path "/d9f7c98a-e535-4a62-9291-f3e87bb98657"
-      (reference "J2") (unit 1) (value "Conn_01x04") (footprint "")
+      (reference "J2") (unit 1) (value "Conn_01x04") (footprint "Connector_PinHeader_2.54mm:PinHeader_1x04_P2.54mm_Vertical")
     )
     (path "/ff7ac0cb-f31b-417e-9005-930a8564c07e"
-      (reference "J3") (unit 1) (value "Conn_01x02") (footprint "")
+      (reference "J3") (unit 1) (value "Conn_01x02") (footprint "Connector_PinHeader_2.54mm:PinHeader_1x02_P2.54mm_Vertical")
     )
   )

Commit message: feat: update artwork
Parts:
- J1: footprint (none) -> Connector_PinHeader_1.27mm:PinHeader_2x05_P1.27mm_Vertical
- J2: footprint (none) -> Connector_PinHeader_2.54mm:PinHeader_1x04_P2.54mm_Vertical
- J3: footprint (none) -> Connector_PinHeader_2.54mm:PinHeader_1x02_P2.54mm_Vertical
Changed lines of the file:
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@@
     (property "Reference" "J1" (id 0) (at 111.125 85.09 0))
     (property "Value" "Conn_02x05_Top_Bottom" (id 1) (at 111.125 87.63 0))
-    (property "Footprint" "" (id 2) (at 109.855 96.52 0)
+    (property "Footprint" "Connector_PinHeader_1.27mm:PinHeader_2x05_P1.27mm_Vertical" (id 2) (at 109.855 96.52 0)
       (effects (font (size 1.27 1.27)) hide)
     )
@@
       (effects (font (size 1.27 1.27)) (justify left))
     )
-    (property "Footprint" "" (id 2) (at 159.385 94.615 0)
+    (property "Footprint" "Connector_PinHeader_2.54mm:PinHeader_1x04_P2.54mm_Vertical" (id 2) (at 159.385 94.615 0)
       (effects (font (size 1.27 1.27)) hide)
     )
@@
       (effects (font (size 1.27 1.27)) (justify left))
     )
-    (property "Footprint" "" (id 2) (at 159.385 112.395 0)
+    (property "Footprint" "Connector_PinHeader_2.54mm:PinHeader_1x02_P2.54mm_Vertical" (id 2) (at 159.385 112.395 0)
       (effects (font (size 1.27 1.27)) hide)
     )

Commit message: feat: update component
Parts:
- J1: footprint Connector_PinHeader_1.27mm:PinHeader_2x05_P1.27mm_Vertical -> (none)
Changed lines of the file:
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@@
     (property "Reference" "J1" (id 0) (at 111.125 85.09 0))
     (property "Value" "Conn_02x05_Top_Bottom" (id 1) (at 111.125 87.63 0))
-    (property "Footprint" "Connector_PinHeader_1.27mm:PinHeader_2x05_P1.27mm_Vertical" (id 2) (at 109.855 96.52 0)
+    (property "Footprint" "" (id 2) (at 109.855 96.52 0)
       (effects (font (size 1.27 1.27)) hide)
     )
@@
     )
     (path "/7269c319-0767-4b85-898a-3b8bb1c1b467"
-      (reference "J1") (unit 1) (value "Conn_02x05_Top_Bottom") (footprint "Connector_PinHeader_1.27mm:PinHeader_2x05_P1.27mm_Vertical")
+      (reference "J1") (unit 1) (value "Conn_02x05_Top_Bottom") (footprint "Connector_PinSocket_1.27mm:PinSocket_2x05_P1.27mm_Vertical")
     )
     (path "/d9f7c98a-e535-4a62-9291-f3e87bb98657"

Commit message: feat: update schematic
Parts:
- J1: value Conn_02x05_Top_Bottom -> (none)
- J2: value Conn_01x04 -> (none); footprint Connector_PinHeader_2.54mm:PinHeader_1x04_P2.54mm_Vertical -> (none)
- J3: value Conn_01x02 -> (none); footprint Connector_PinHeader_2.54mm:PinHeader_1x02_P2.54mm_Vertical -> (none)
Changed lines of the file:
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@@
     (in_bom yes) (on_board yes) (fields_autoplaced)
     (property "Reference" "J1" (id 0) (at 111.125 85.09 0))
-    (property "Value" "Conn_02x05_Top_Bottom" (id 1) (at 111.125 87.63 0))
+    (property "Value" "" (id 1) (at 111.125 87.63 0))
     (property "Footprint" "" (id 2) (at 109.855 96.52 0)
       (effects (font (size 1.27 1.27)) hide)
@@
       (effects (font (size 1.27 1.27)) (justify left))
     )
-    (property "Value" "Conn_01x04" (id 1) (at 162.56 97.1549 0)
+    (property "Value" "" (id 1) (at 162.56 97.1549 0)
       (effects (font (size 1.27 1.27)) (justify left))
     )
-    (property "Footprint" "Connector_PinHeader_2.54mm:PinHeader_1x04_P2.54mm_Vertical" (id 2) (at 159.385 94.615 0)
+    (property "Footprint" "" (id 2) (at 159.385 94.615 0)
       (effects (font (size 1.27 1.27)) hide)
     )
@@
       (effects (font (size 1.27 1.27)) (justify left))
     )
-    (property "Value" "Conn_01x02" (id 1) (at 162.56 114.9349 0)
+    (property "Value" "" (id 1) (at 162.56 114.9349 0)
       (effects (font (size 1.27 1.27)) (justify left))
     )
-    (property "Footprint" "Connector_PinHeader_2.54mm:PinHeader_1x02_P2.54mm_Vertical" (id 2) (at 159.385 112.395 0)
+    (property "Footprint" "" (id 2) (at 159.385 112.395 0)
       (effects (font (size 1.27 1.27)) hide)
     )
